File: canvas/routing_template/touch_probe/touch_probe/touch_probe.kicad_pcb (KiCad board)
At the start: 2 copper layers, 90 x 15 mm, 4 parts, among them J1 Conn_01x01, J2 Conn_01x01, J3 Conn_01x01, J4 Conn_01x01

Commit message: SUKU touch_probe done
Other:
- board size 90 x 15 mm -> 71.5 x 14.5 mm
- board text added: "NO SOLDERMASK AND SILCSCREEN ON PCB JUST GOLD PLATED COPPER"
Changed lines of the file:
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@@
   (general
     (thickness 1.6)
-    (drawings 34)
+    (drawings 25)
     (tracks 0)
     (zones 0)
@@
     (aux_axis_origin 100 100)
     (grid_origin 100 100)
-    (visible_elements FFFFFF7F)
+    (visible_elements 7FFFFFFF)
     (pcbplotparams
-      (layerselection 0x010fc_ffffffff)
+      (layerselection 0x010f0_ffffffff)
       (usegerberextensions false)
       (usegerberattributes true)
@@
       (outputformat 1)
       (mirror false)
-      (drillshape 1)
+      (drillshape 0)
       (scaleselection 1)
-      (outputdirectory ""))
+      (outputdirectory "mfg/"))
   )
   (net 0 "")
@@
       (net 1 GND))
   )
+  (gr_text "NO SOLDERMASK AND SILCSCREEN ON PCB\nJUST GOLD PLATED COPPER" (at 100 94.5) (layer F.SilkS)
+    (effects (font (size 1 1) (thickness 0.15)))
+  )
+  (gr_line (start 135.75 114.5) (end 135.75 100) (layer Edge.Cuts) (width 0.05))
+  (gr_line (start 64.25 114.5) (end 135.75 114.5) (layer Edge.Cuts) (width 0.05))
+  (gr_line (start 64.25 100) (end 64.25 114.5) (layer Edge.Cuts) (width 0.05))
   (gr_poly (pts (xy 147 117) (xy 53 117) (xy 53 98) (xy 147 98)) (layer B.Mask) (width 0.1))
   (gr_poly (pts (xy 147 117) (xy 53 117) (xy 53 98) (xy 147 98)) (layer F.Mask) (width 0.1))
   (gr_arc (start 107 109) (end 107 110) (angle -90) (layer Edge.Cuts) (width 0.05))
   (gr_arc (start 93 109) (end 92 109) (angle -90) (layer Edge.Cuts) (width 0.05))
-  (gr_line (start 141.005 104) (end 141.005 100) (layer Edge.Cuts) (width 0.05))
-  (gr_line (start 139.005 104) (end 139.005 100) (layer Edge.Cuts) (width 0.05))
-  (gr_line (start 114.335 104) (end 114.335 100) (layer Edge.Cuts) (width 0.05))
-  (gr_line (start 112.335 104) (end 112.335 100) (layer Edge.Cuts) (width 0.05))
-  (gr_line (start 87.665 104) (end 87.665 100) (layer Edge.Cuts) (width 0.05))
-  (gr_line (start 85.665 104) (end 85.665 100) (layer Edge.Cuts) (width 0.05))
-  (gr_line (start 60.995 104) (end 60.995 100) (layer Edge.Cuts) (width 0.05))
-  (gr_line (start 58.995 104) (end 58.995 100) (layer Edge.Cuts) (width 0.05))
-  (gr_line (start 108 100) (end 112.335 100) (layer Edge.Cuts) (width 0.05))
+  (gr_line (start 114.835 104) (end 114.835 100) (layer Edge.Cuts) (width 0.05))
+  (gr_line (start 111.835 104) (end 111.835 100) (layer Edge.Cuts) (width 0.05))
+  (gr_line (start 88.165 104) (end 88.165 100) (layer Edge.Cuts) (width 0.05))
+  (gr_line (start 85.165 104) (end 85.165 100) (layer Edge.Cuts) (width 0.05))
+  (gr_line (start 108 100) (end 111.835 100) (layer Edge.Cuts) (width 0.05))
   (gr_line (start 108 109) (end 108 100) (layer Edge.Cuts) (width 0.05))
   (gr_line (start 93 110) (end 107 110) (layer Edge.Cuts) (width 0.05))
   (gr_line (start 92 100) (end 92 109) (layer Edge.Cuts) (width 0.05))
-  (gr_line (start 87.665 100) (end 92 100) (layer Edge.Cuts) (width 0.05))
-  (gr_line (start 141.005 100) (end 145 100) (layer Edge.Cuts) (width 0.05))
-  (gr_line (start 114.335 100) (end 139.005 100) (layer Edge.Cuts) (width 0.05))
-  (gr_line (start 60.995 100) (end 85.665 100) (layer Edge.Cuts) (width 0.05))
-  (gr_arc (start 59.995 104) (end 58.995 104) (angle -180) (layer Edge.Cuts) (width 0.05))
-  (gr_arc (start 140.005 104) (end 139.005 104) (angle -180) (layer Edge.Cuts) (width 0.05))
-  (gr_arc (start 113.335 104) (end 112.335 104) (angle -180) (layer Edge.Cuts) (width 0.05))
-  (gr_arc (start 86.665 104) (end 85.665 104) (angle -180) (layer Edge.Cuts) (width 0.05))
-  (gr_line (start 59.995 100) (end 59.995 95) (layer Dwgs.User) (width 0.15))
-  (gr_line (start 140.005 100) (end 140.005 95) (layer Dwgs.User) (width 0.15))
+  (gr_line (start 88.165 100) (end 92 100) (layer Edge.Cuts) (width 0.05))
+  (gr_line (start 114.835 100) (end 135.75 100) (layer Edge.Cuts) (width 0.05))
+  (gr_line (start 64.25 100) (end 85.165 100) (layer Edge.Cuts) (width 0.05))
+  (gr_arc (start 113.335 104) (end 111.835 104) (angle -180) (layer Edge.Cuts) (width 0.05))
+  (gr_arc (start 86.665 104) (end 85.165 104) (angle -180) (layer Edge.Cuts) (width 0.05))
   (gr_line (start 113.335 100) (end 113.335 95) (layer Dwgs.User) (width 0.15))
   (gr_line (start 86.665 100) (end 86.665 95) (layer Dwgs.User) (width 0.15))
   (gr_line (start 126.67 100) (end 126.67 90) (layer Dwgs.User) (width 0.15))
   (gr_line (start 73.33 100) (end 73.33 90) (layer Dwgs.User) (width 0.15))
-  (gr_line (start 55 100) (end 58.995 100) (layer Edge.Cuts) (width 0.05))
-  (gr_line (start 145 115) (end 145 100) (layer Edge.Cuts) (width 0.05))
-  (gr_line (start 55 115) (end 145 115) (layer Edge.Cuts) (width 0.05))
-  (gr_line (start 55 100) (end 55 115) (layer Edge.Cuts) (width 0.05))
   (zone (net 1) (net_name GND) (layer F.Cu) (hatch edge 0.508)
     (connect_pads yes (clearance 0.25))
